File: cd32/eagle/cd32.sch (EAGLE design)
At the start: 2 parts, among them CN1 CD32-EXPANSION, CN2 CD32-EXPANSION

Commit message: updates.. adjusted board shape... not finished yet Added Maxim RS232 chip
Parts:
- added C1, C2, C3: (no value), eagle-ltspice:CC1206
- added IC1: MAX3311, maxim:MAX3311
Connections:
- new net GND: C3.2, IC1.GND
- new net N$1: C1.1, IC1.C1+
- new net N$2: C1.2, IC1.C1-
- new net N$3: C2.1, IC1.V-
- new net VCC: C3.1, IC1.VCC
- net +12V@1: now also C2.2
- net _RXD: now also IC1.ROUT
- net _TXD: now also IC1.TIN
Changed lines of the file:
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@@
 <layer number="54" name="bGND_GNDA" color="7" fill="1" visible="no" active="no"/>
 <layer number="56" name="wert" color="7" fill="1" visible="no" active="no"/>
+<layer number="57" name="tCAD" color="7" fill="1" visible="no" active="no"/>
+<layer number="59" name="tCarbon" color="7" fill="1" visible="no" active="no"/>
+<layer number="60" name="bCarbon" color="7" fill="1" visible="no" active="no"/>
 <layer number="90" name="Modules" color="5" fill="1" visible="yes" active="yes"/>
 <layer number="91" name="Nets" color="2" fill="1" visible="yes" active="yes"/>
@@
 <layer number="97" name="Info" color="7" fill="1" visible="yes" active="yes"/>
 <layer number="98" name="Guide" color="6" fill="1" visible="yes" active="yes"/>
+<layer number="99" name="SpiceOrder" color="7" fill="1" visible="no" active="no"/>
 <layer number="100" name="Muster" color="7" fill="1" visible="yes" active="yes"/>
 <layer number="101" name="Patch_Top" color="7" fill="1" visible="yes" active="yes"/>
@@
 <layer number="106" name="bPlate" color="7" fill="1" visible="yes" active="yes"/>
 <layer number="107" name="Crop" color="7" fill="1" visible="yes" active="yes"/>
+<layer number="108" name="tplace-old" color="10" fill="1" visible="yes" active="yes"/>
+<layer number="109" name="ref-old" color="11" fill="1" visible="yes" active="yes"/>
 <layer number="110" name="tdokum" color="7" fill="1" visible="yes" active="yes"/>
 <layer number="111" name="bdokum" color="7" fill="1" visible="yes" active="yes"/>
+<layer number="112" name="tSilk" color="7" fill="1" visible="yes" active="yes"/>
+<layer number="113" name="IDFDebug" color="4" fill="1" visible="yes" active="yes"/>
+<layer number="114" name="Badge_Outline" color="7" fill="1" visible="yes" active="yes"/>
+<layer number="115" name="ReferenceISLANDS" color="7" fill="1" visible="yes" active="yes"/>
 <layer number="116" name="Patch_BOT" color="7" fill="1" visible="yes" active="yes"/>
+<layer number="118" name="Rect_Pads" color="7" fill="1" visible="yes" active="yes"/>
 <layer number="121" name="_tsilk" color="7" fill="1" visible="yes" active="yes"/>
 <layer number="122" name="_bsilk" color="7" fill="1" visible="yes" active="yes"/>
+<layer number="123" name="tTestmark" color="7" fill="1" visible="yes" active="yes"/>
+<layer number="124" name="bTestmark" color="7" fill="1" visible="yes" active="yes"/>
+<layer number="125" name="_tNames" color="7" fill="1" visible="yes" active="yes"/>
+<layer number="126" name="_bNames" color="7" fill="1" visible="yes" active="yes"/>
+<layer number="127" name="_tValues" color="7" fill="1" visible="yes" active="yes"/>
+<layer number="128" name="_bValues" color="7" fill="1" visible="yes" active="yes"/>
+<layer number="129" name="Mask" color="7" fill="1" visible="yes" active="yes"/>
+<layer number="131" name="tAdjust" color="7" fill="1" visible="yes" active="yes"/>
+<layer number="132" name="bAdjust" color="7" fill="1" visible="yes" active="yes"/>
+<layer number="144" name="Drill_legend" color="7" fill="1" visible="yes" active="yes"/>
+<layer number="150" name="Notes" color="7" fill="1" visible="yes" active="yes"/>
 <layer number="151" name="HeatSink" color="7" fill="1" visible="yes" active="yes"/>
+<layer number="152" name="_bDocu" color="7" fill="1" visible="yes" active="yes"/>
+<layer number="153" name="FabDoc1" color="7" fill="1" visible="yes" active="yes"/>
+<layer number="154" name="FabDoc2" color="7" fill="1" visible="yes" active="yes"/>
+<layer number="155" name="FabDoc3" color="7" fill="1" visible="yes" active="yes"/>
 <layer number="199" name="Contour" color="7" fill="1" visible="yes" active="yes"/>
 <layer number="200" name="200bmp" color="7" fill="1" visible="yes" active="yes"/>
@@
 <layer number="209" name="209bmp" color="7" fill="1" visible="yes" active="yes"/>
 <layer number="210" name="210bmp" color="7" fill="1" visible="yes" active="yes"/>
+<layer number="211" name="211bmp" color="7" fill="1" visible="yes" active="yes"/>
+<layer number="212" name="212bmp" color="7" fill="1" visible="yes" active="yes"/>
+<layer number="213" name="213bmp" color="7" fill="1" visible="yes" active="yes"/>
+<layer number="214" name="214bmp" color="7" fill="1" visible="yes" active="yes"/>
+<layer number="215" name="215bmp" color="7" fill="1" visible="yes" active="yes"/>
+<layer number="216" name="216bmp" color="7" fill="1" visible="yes" active="yes"/>
+<layer number="217" name="217bmp" color="18" fill="1" visible="no" active="no"/>
+<layer number="218" name="218bmp" color="19" fill="1" visible="no" active="no"/>
+<layer number="219" name="219bmp" color="20" fill="1" visible="no" active="no"/>
+<layer number="220" name="220bmp" color="21" fill="1" visible="no" active="no"/>
+<layer number="221" name="221bmp" color="22" fill="1" visible="no" active="no"/>
+<layer number="222" name="222bmp" color="23" fill="1" visible="no" active="no"/>
+<layer number="223" name="223bmp" color="24" fill="1" visible="no" active="no"/>
+<layer number="224" name="224bmp" color="25" fill="1" visible="no" active="no"/>
+<layer number="225" name="225bmp" color="7" fill="1" visible="yes" active="yes"/>
+<layer number="226" name="226bmp" color="7" fill="1" visible="yes" active="yes"/>
+<layer number="227" name="227bmp" color="7" fill="1" visible="yes" active="yes"/>
+<layer number="228" name="228bmp" color="7" fill="1" visible="yes" active="yes"/>
+<layer number="229" name="229bmp" color="7" fill="1" visible="yes" active="yes"/>
+<layer number="230" name="230bmp" color="7" fill="1" visible="yes" active="yes"/>
+<layer number="231" name="231bmp" color="7" fill="1" visible="yes" active="yes"/>
 <layer number="248" name="PLCDoku" color="7" fill="1" visible="yes" active="yes"/>
 <layer number="249" name="MillDoku" color="7" fill="1" visible="yes" active="yes"/>
@@
 <part name="CN1" library="Amiga" deviceset="CD32-EXPANSION" device=""/>
 <part name="CN2" library="Amiga" deviceset="CD32-EXPANSION" device=""/>
+<part name="IC1" library="maxim" deviceset="MAX3311" device=""/>
+<part name="C1" library="eagle-ltspice" deviceset="C" device="C1206"/>
+<part name="C2" library="eagle-ltspice" deviceset="C" device="C1206"/>
+<part name="C3" library="eagle-ltspice" deviceset="C" device="C1206"/>
 </parts>
 <sheets>
@@
 <instance part="CN1" gate="CD32_EXPANSION" x="101.6" y="154.94"/>
 <instance part="CN2" gate="CD32_EXPANSION" x="304.8" y="154.94"/>
+<instance part="IC1" gate="G$1" x="434.34" y="114.3"/>
+<instance part="C1" gate="G$1" x="459.74" y="119.38"/>
+<instance part="C2" gate="G$1" x="462.28" y="101.6"/>
+<instance part="C3" gate="G$1" x="474.98" y="119.38"/>
 </instances>
 <busses>
@@
 <label x="242.57" y="99.06" size="1.778" layer="95"/>
 </segment>
+<segment>
+<pinref part="IC1" gate="G$1" pin="ROUT"/>
+<wire x1="406.4" y1="109.22" x2="421.64" y2="109.22" width="0.1524" layer="91"/>
+</segment>
 </net>
 <net name="+12V@1" class="0">
@@
 <wire x1="327.66" y1="88.9" x2="406.4" y2="88.9" width="0.1534" layer="91"/>
 <label x="367.03" y="88.9" size="1.778" layer="95"/>
+<pinref part="C2" gate="G$1" pin="2"/>
+<wire x1="406.4" y1="88.9" x2="462.28" y2="88.9" width="0.1524" layer="91"/>
+<wire x1="462.28" y1="88.9" x2="462.28" y2="96.52" width="0.1524" layer="91"/>
 </segment>
 </net>
@@
 <label x="367.03" y="99.06" size="1.778" layer="95"/>
 </segment>
+<segment>
+<pinref part="IC1" gate="G$1" pin="TIN"/>
+<wire x1="406.4" y1="111.76" x2="421.64" y2="111.76" width="0.1524" layer="91"/>
+</segment>
 </net>
 <net name="NC@9" class="0">
@@
 </segment>
 </net>
+<net name="VCC" class="0">
+<segment>
+<pinref part="IC1" gate="G$1" pin="VCC"/>
+<wire x1="406.4" y1="121.92" x2="416.56" y2="121.92" width="0.1524" layer="91"/>
+<wire x1="416.56" y1="121.92" x2="421.64" y2="121.92" width="0.1524" layer="91"/>
+<wire x1="416.56" y1="121.92" x2="416.56" y2="132.08" width="0.1524" layer="91"/>
+<wire x1="416.56" y1="132.08" x2="474.98" y2="132.08" width="0.1524" layer="91"/>
+<pinref part="C3" gate="G$1" pin="1"/>
+<wire x1="474.98" y1="132.08" x2="474.98" y2="121.92" width="0.1524" layer="91"/>
+</segment>
+</net>
+<net name="GND" class="0">
+<segment>
+<pinref part="IC1" gate="G$1" pin="GND"/>
+<wire x1="406.4" y1="104.14" x2="421.64" y2="104.14" width="0.1524" layer="91"/>
+</segment>
+<segment>
+<pinref part="C3" gate="G$1" pin="2"/>
+<wire x1="406.4" y1="81.28" x2="474.98" y2="81.28" width="0.1524" layer="91"/>
+<wire x1="474.98" y1="81.28" x2="474.98" y2="114.3" width="0.1524" layer="91"/>
+</segment>
+</net>
+<net name="N$1" class="0">
+<segment>
+<pinref part="IC1" gate="G$1" pin="C1+"/>
+<pinref part="C1" gate="G$1" pin="1"/>
+<wire x1="447.04" y1="121.92" x2="459.74" y2="121.92" width="0.1524" layer="91"/>
+</segment>
+</net>
+<net name="N$2" class="0">
+<segment>
+<pinref part="IC1" gate="G$1" pin="C1-"/>
+<pinref part="C1" gate="G$1" pin="2"/>
+<wire x1="447.04" y1="116.84" x2="447.04" y2="114.3" width="0.1524" layer="91"/>
+<wire x1="447.04" y1="114.3" x2="459.74" y2="114.3" width="0.1524" layer="91"/>
+</segment>
+</net>
+<net name="N$3" class="0">
+<segment>
+<pinref part="IC1" gate="G$1" pin="V-"/>
+<pinref part="C2" gate="G$1" pin="1"/>
+<wire x1="447.04" y1="104.14" x2="462.28" y2="104.14" width="0.1524" layer="91"/>
+</segment>
+</net>
